File: poweramp.kicad_sch (KiCad schematic)
At the start: 81 parts, among them IC1 TPA3255, U2 Opamp_Dual

Commit message: add bypass caps to opamps + swap poweramps + layout progress
Parts:
- added CU2: 10u, invendelirium_audio:C_0603, symbol Device:C
- C14: value 10u -> 1uF
Connections:
- net 12V: now also CU2.1
- net GND: now also CU2.2
Other:
- moved on the sheet: U2C
Changed lines of the file:
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@@
   (junction (at 241.3 123.19) (diameter 0) (color 0 0 0 0)
   )
+  (junction (at 191.77 162.56) (diameter 0) (color 0 0 0 0)
+  )
   (junction (at 233.68 123.19) (diameter 0) (color 0 0 0 0)
   )
@@
     (stroke (width 0) (type default))
   )
+  (wire (pts (xy 191.77 147.32) (xy 210.82 147.32))
+    (stroke (width 0) (type default))
+  )
   (wire (pts (xy 241.3 110.49) (xy 251.46 110.49))
     (stroke (width 0) (type default))
@@
     (stroke (width 0) (type default))
   )
+  (wire (pts (xy 210.82 147.32) (xy 210.82 151.13))
+    (stroke (width 0) (type default))
+  )
   (wire (pts (xy 85.09 125.73) (xy 87.63 125.73))
     (stroke (width 0) (type default))
@@
     (stroke (width 0) (type default))
   )
+  (wire (pts (xy 210.82 158.75) (xy 210.82 162.56))
+    (stroke (width 0) (type default))
+  )
   (wire (pts (xy 52.07 177.8) (xy 58.42 177.8))
     (stroke (width 0) (type default))
@@
     (stroke (width 0) (type default))
   )
+  (wire (pts (xy 191.77 162.56) (xy 210.82 162.56))
+    (stroke (width 0) (type default))
+  )
   (wire (pts (xy 104.14 62.23) (xy 107.95 62.23))
     (stroke (width 0) (type default))
@@
     (effects (font (size 1.27 1.27)) (justify left bottom))
   )
-  (label "12V" (at 163.83 177.8 0) (fields_autoplaced)
+  (label "12V" (at 194.31 147.32 0) (fields_autoplaced)
     (effects (font (size 1.27 1.27)) (justify left bottom))
   )
@@
       (effects (font (size 1.27 1.27)) (justify left))
     )
-    (property "Value" "10u" (at 78.74 106.68 0)
+    (property "Value" "1uF" (at 78.74 106.68 0)
       (effects (font (size 1.27 1.27)) (justify left))
     )
@@
     )
   )
+  (symbol (lib_id "Device:C") (at 210.82 154.94 0) (unit 1)
+    (in_bom yes) (on_board yes) (dnp no)
+    (property "Reference" "CU2" (at 212.09 152.4 0)
+      (effects (font (size 1.27 1.27)) (justify left))
+    )
+    (property "Value" "10u" (at 212.09 157.48 0)
+      (effects (font (size 1.27 1.27)) (justify left))
+    )
+    (property "Footprint" "invendelirium_audio:C_0603" (at 211.7852 158.75 0)
+      (effects (font (size 1.27 1.27)) hide)
+    )
+    (property "Datasheet" "~" (at 210.82 154.94 0)
+      (effects (font (size 1.27 1.27)) hide)
+    )
+    (property "Voltage" "16V" (at 210.82 154.94 0)
+      (effects (font (size 1.27 1.27)) hide)
+    )
+    (pin "1")
+    (pin "2")
+    (instances
+      (project "uberamp1"
+        (path "/310059c1-d84b-43e2-9c9a-0e426c534a12/5156a0a1-195e-40e3-846d-487893ba8fa7"
+          (reference "CU2") (unit 1)
+        )
+        (path "/310059c1-d84b-43e2-9c9a-0e426c534a12/f0f90934-0ffc-42c4-856c-3b886cd79d06"
+          (reference "CU3") (unit 1)
+        )
+      )
+    )
+  )
   (symbol (lib_id "Device:C") (at 77.47 127 0) (unit 1)
     (in_bom yes) (on_board yes) (dnp no) (fields_autoplaced)
@@
     )
   )
-  (symbol (lib_id "Device:Opamp_Dual") (at 166.37 185.42 0) (unit 3)
+  (symbol (lib_id "Device:Opamp_Dual") (at 194.31 154.94 0) (unit 3)
     (in_bom yes) (on_board yes) (dnp no) (fields_autoplaced)
-    (property "Reference" "U2" (at 165.1 184.785 0)
+    (property "Reference" "U2" (at 193.04 154.305 0)
       (effects (font (size 1.27 1.27)) (justify left))
     )
-    (property "Value" "Opamp_Dual" (at 165.1 187.325 0)
+    (property "Value" "Opamp_Dual" (at 193.04 156.845 0)
       (effects (font (size 1.27 1.27)) (justify left))
     )
-    (property "Footprint" "invendelirium_audio:SOIC-8" (at 166.37 185.42 0)
+    (property "Footprint" "invendelirium_audio:SOIC-8" (at 194.31 154.94 0)
       (effects (font (size 1.27 1.27)) hide)
     )
-    (property "Datasheet" "~" (at 166.37 185.42 0)
+    (property "Datasheet" "~" (at 194.31 154.94 0)
       (effects (font (size 1.27 1.27)) hide)
     )
@@
     )
   )
-  (symbol (lib_id "power:GND") (at 163.83 193.04 0) (unit 1)
+  (symbol (lib_id "power:GND") (at 191.77 162.56 0) (unit 1)
     (in_bom yes) (on_board yes) (dnp no) (fields_autoplaced)
-    (property "Reference" "#PWR011" (at 163.83 199.39 0)
+    (property "Reference" "#PWR011" (at 191.77 168.91 0)
       (effects (font (size 1.27 1.27)) hide)
     )
-    (property "Value" "GND" (at 163.83 198.12 0)
+    (property "Value" "GND" (at 191.77 167.64 0)
       (effects (font (size 1.27 1.27)) hide)
     )
-    (property "Footprint" "" (at 163.83 193.04 0)
+    (property "Footprint" "" (at 191.77 162.56 0)
       (effects (font (size 1.27 1.27)) hide)
     )
-    (property "Datasheet" "" (at 163.83 193.04 0)
+    (property "Datasheet" "" (at 191.77 162.56 0)
       (effects (font (size 1.27 1.27)) hide)
     )

Commit message: add bypass caps to fakegnd
Parts:
- added CR0: 10u, invendelirium_audio:C_0603, symbol Device:C
Connections:
- net GND: now also CR0.2
- net input_ref: now also CR0.1
Changed lines of the file:
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@@
   (junction (at 175.26 92.71) (diameter 0) (color 0 0 0 0)
   )
+  (junction (at 166.37 149.86) (diameter 0) (color 0 0 0 0)
+  )
   (junction (at 181.61 105.41) (diameter 0) (color 0 0 0 0)
   )
@@
     (stroke (width 0) (type default))
   )
-  (wire (pts (xy 162.56 149.86) (xy 163.83 149.86))
-    (stroke (width 0) (type default))
-  )
   (wire (pts (xy 179.07 77.47) (xy 170.18 77.47))
     (stroke (width 0) (type default))
@@
     (stroke (width 0) (type default))
   )
+  (wire (pts (xy 162.56 149.86) (xy 166.37 149.86))
+    (stroke (width 0) (type default))
+  )
   (wire (pts (xy 170.18 90.17) (xy 175.26 90.17))
     (stroke (width 0) (type default))
@@
     (stroke (width 0) (type default))
   )
+  (wire (pts (xy 166.37 149.86) (xy 171.45 149.86))
+    (stroke (width 0) (type default))
+  )
   (wire (pts (xy 186.69 115.57) (xy 194.31 115.57))
     (stroke (width 0) (type default))
@@
     (effects (font (size 1.27 1.27)) (justify right))
   )
-  (hierarchical_label "input_ref" (shape output) (at 163.83 149.86 0) (fields_autoplaced)
+  (hierarchical_label "input_ref" (shape output) (at 171.45 149.86 0) (fields_autoplaced)
     (effects (font (size 1.27 1.27)) (justify left))
   )
@@
     )
   )
+  (symbol (lib_id "Device:C") (at 166.37 153.67 0) (unit 1)
+    (in_bom yes) (on_board yes) (dnp no)
+    (property "Reference" "CR0" (at 167.64 151.13 0)
+      (effects (font (size 1.27 1.27)) (justify left))
+    )
+    (property "Value" "10u" (at 167.64 156.21 0)
+      (effects (font (size 1.27 1.27)) (justify left))
+    )
+    (property "Footprint" "invendelirium_audio:C_0603" (at 167.3352 157.48 0)
+      (effects (font (size 1.27 1.27)) hide)
+    )
+    (property "Datasheet" "~" (at 166.37 153.67 0)
+      (effects (font (size 1.27 1.27)) hide)
+    )
+    (property "Voltage" "16V" (at 166.37 153.67 0)
+      (effects (font (size 1.27 1.27)) hide)
+    )
+    (pin "1")
+    (pin "2")
+    (instances
+      (project "uberamp1"
+        (path "/310059c1-d84b-43e2-9c9a-0e426c534a12/5156a0a1-195e-40e3-846d-487893ba8fa7"
+          (reference "CR0") (unit 1)
+        )
+        (path "/310059c1-d84b-43e2-9c9a-0e426c534a12/f0f90934-0ffc-42c4-856c-3b886cd79d06"
+          (reference "CR1") (unit 1)
+        )
+      )
+    )
+  )
   (symbol (lib_id "Device:R_Small") (at 118.11 132.08 270) (unit 1)
     (in_bom yes) (on_board yes) (dnp no)
@@
         )
       )
+    )
+  )
+  (symbol (lib_id "power:GND") (at 166.37 157.48 0) (unit 1)
+    (in_bom yes) (on_board yes) (dnp no) (fields_autoplaced)
+    (property "Reference" "#PWR084" (at 166.37 163.83 0)
+      (effects (font (size 1.27 1.27)) hide)
+    )
+    (property "Value" "GND" (at 166.37 162.56 0)
+      (effects (font (size 1.27 1.27)) hide)
+    )
+    (property "Footprint" "" (at 166.37 157.48 0)
+      (effects (font (size 1.27 1.27)) hide)
+    )
+    (property "Datasheet" "" (at 166.37 157.48 0)
+      (effects (font (size 1.27 1.27)) hide)
+    )
+    (pin "1")
+    (instances
+      (project "uberamp1"
+        (path "/310059c1-d84b-43e2-9c9a-0e426c534a12/5156a0a1-195e-40e3-846d-487893ba8fa7"
+          (reference "#PWR084") (unit 1)
+        )
+        (path "/310059c1-d84b-43e2-9c9a-0e426c534a12/f0f90934-0ffc-42c4-856c-3b886cd79d06"
+          (reference "#PWR085") (unit 1)
+        )
+      )

Commit message: minor schematic updates
Other:
- note added: "3.82V"
Changed lines of the file:
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@@
     (stroke (width 0) (type default))
+  )
+  (text "3.82V" (at 166.37 148.59 0)
+    (effects (font (size 1.016 1.016)) (justify left bottom))
   )
   (text "4.54vpp" (at 60.96 157.48 0)

Commit message: schematic: some fixes
Parts:
- added s30: reset, invendelirium_general:pad_1.2x1.5, symbol Connector:TestPoint
Connections:
- net ~reset: now also s30.1
Changed lines of the file:
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@@
 	)
 	(junction
+		(at 41.91 128.27)
+		(diameter 0)
+		(color 0 0 0 0)
+	)
+	(junction
 		(at 123.19 190.5)
 		(diameter 0)
@@
 	(wire
 		(pts
-			(xy 43.18 128.27) (xy 45.72 128.27)
-		)
-		(stroke
-			(width 0)
-			(type default)
-		)
-	)
-	(wire
-		(pts
 			(xy 233.68 92.71) (xy 241.3 92.71)
 		)
@@
 	(wire
 		(pts
+			(xy 38.1 128.27) (xy 41.91 128.27)
+		)
+		(stroke
+			(width 0)
+			(type default)
+		)
+	)
+	(wire
+		(pts
 			(xy 175.26 59.69) (xy 179.07 59.69)
 		)
@@
 	(wire
 		(pts
+			(xy 41.91 128.27) (xy 45.72 128.27)
+		)
+		(stroke
+			(width 0)
+			(type default)
+		)
+	)
+	(wire
+		(pts
 			(xy 162.56 157.48) (xy 162.56 149.86)
 		)
@@
 	(hierarchical_label "~reset"
 		(shape input)
-		(at 44.45 128.27 180)
+		(at 38.1 128.27 180)
 		(fields_autoplaced yes)
 		(effects
@@
 					(unit 1)
 				)
+			)
+		)
+	)
+	(symbol
+		(lib_id "Connector:TestPoint")
+		(at 41.91 128.27 0)
+		(unit 1)
+		(exclude_from_sim no)
+		(in_bom yes)
+		(on_board yes)
+		(dnp no)
+		(property "Reference" "s30"
+			(at 40.64 120.65 0)
+			(effects
+				(font
+					(size 1.27 1.27)
+				)
+				(justify left)
+			)
+		)
+		(property "Value" "reset"
+			(at 40.64 121.92 0)
+			(effects
+				(font
+					(size 1.27 1.27)
+				)
+				(justify left)
+			)
+		)
+		(property "Footprint" "invendelirium_general:pad_1.2x1.5"
+			(at 46.99 128.27 0)
+			(effects
+				(font
+					(size 1.27 1.27)
+				)
+				(hide yes)
+			)
+		)
+		(property "Datasheet" "~"
+			(at 46.99 128.27 0)
+			(effects
+				(font
+					(size 1.27 1.27)
+				)
+				(hide yes)
+			)
+		)
+		(property "Description" ""
+			(at 41.91 128.27 0)
+			(effects
+				(font
+					(size 1.27 1.27)
+				)
+				(hide yes)
+			)
+		)
+		(pin "1"
+		)
+		(instances
+			(project "uberamp1"
+				(path "/310059c1-d84b-43e2-9c9a-0e426c534a12/5156a0a1-195e-40e3-846d-487893ba8fa7"
+					(reference "s30")
+					(unit 1)
+				)
+				(path "/310059c1-d84b-43e2-9c9a-0e426c534a12/f0f90934-0ffc-42c4-856c-3b886cd79d06"
+					(reference "s31")
+					(unit 1)
+				)

Commit message: add power input +...
+ tons of fixes, footprint assignments, etc
Parts:
- C23, C24, C25, C26: PN (none) -> CL32B106KMVNNWE

Commit message: update some footprints
Parts:
- D1, D2, D3, D4, D5, D6, D7, D8: footprint Diode_SMD:D_0805_2012Metric -> invendelirium_general:D_0805
- LED1, LED2: footprint LED_SMD:LED_0805_2012Metric -> invendelirium_general:D_0805
Changed lines of the file:
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@@
 			)
 		)
-		(property "Footprint" "Diode_SMD:D_0805_2012Metric"
+		(property "Footprint" "invendelirium_general:D_0805"
 			(at 241.3 96.52 0)
 			(effects
@@
 			)
 		)
-		(property "Footprint" "Diode_SMD:D_0805_2012Metric"
+		(property "Footprint" "invendelirium_general:D_0805"
 			(at 233.68 114.3 0)
 			(effects
@@
 			)
 		)
-		(property "Footprint" "Diode_SMD:D_0805_2012Metric"
+		(property "Footprint" "invendelirium_general:D_0805"
 			(at 241.3 127 0)
 			(effects
@@
 			)
 		)
-		(property "Footprint" "LED_SMD:LED_0805_2012Metric"
+		(property "Footprint" "invendelirium_general:D_0805"
 			(at 87.63 135.89 0)
 			(effects
@@
 			)
 		)
-		(property "Footprint" "Diode_SMD:D_0805_2012Metric"
+		(property "Footprint" "invendelirium_general:D_0805"
 			(at 233.68 96.52 0)
 			(effects
@@
 			)
 		)
-		(property "Footprint" "Diode_SMD:D_0805_2012Metric"
+		(property "Footprint" "invendelirium_general:D_0805"
 			(at 233.68 127 0)
 			(effects
@@
 			)
 		)
-		(property "Footprint" "LED_SMD:LED_0805_2012Metric"
+		(property "Footprint" "invendelirium_general:D_0805"
 			(at 63.5 130.81 0)
 			(effects
@@
 			)
 		)
-		(property "Footprint" "Diode_SMD:D_0805_2012Metric"
+		(property "Footprint" "invendelirium_general:D_0805"
 			(at 241.3 114.3 0)
 			(effects
@@
 			)
 		)
-		(property "Footprint" "Diode_SMD:D_0805_2012Metric"
+		(property "Footprint" "invendelirium_general:D_0805"
 			(at 241.3 80.01 0)
 			(effects
@@
 			)
 		)
-		(property "Footprint" "Diode_SMD:D_0805_2012Metric"
+		(property "Footprint" "invendelirium_general:D_0805"
 			(at 233.68 80.01 0)
 			(effects

Commit message: fill in some part numbers
Parts:
- C14: value 1uF -> 1u
- C27, C28, C29, C30: PN (none) -> CB052D0105KBC
- C31, C32, C33, C34: value 10nF -> 10nF 63V; PN (none) -> C0603X103K2RECTU
- D1, D2, D3, D4, D5, D6, D7, D8: PN (none) -> RBR1VWM60ATR
- IC1: PN (none) -> TPA3255DDVR
- JP1, JP2, JP3, TP1, TP2, TP3, TP4, s30: now left out of the parts list
- L1, L2, L3, L4: PN (none) -> SPM12565VT-100M-D
- RV1: PN (none) -> TC33X-2-103E
Changed lines of the file:
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@@
 			)
 		)
+		(property "PN" "RBR1VWM60ATR "
+			(at 241.3 96.52 0)
+			(effects
+				(font
+					(size 1.27 1.27)
+				)
+				(hide yes)
+			)
+		)
 		(pin "1"
 		)
@@
 			)
 		)
-		(property "Value" "1uF"
+		(property "Value" "1u"
 			(at 78.74 106.68 0)
 			(effects
@@
 			)
 		)
+		(property "PN" "CB052D0105KBC"
+			(at 208.28 114.3 0)
+			(effects
+				(font
+					(size 1.27 1.27)
+				)
+				(hide yes)
+			)
+		)
 		(pin "1"
 		)
@@
 			)
 		)
+		(property "PN" "RBR1VWM60ATR "
+			(at 233.68 114.3 0)
+			(effects
+				(font
+					(size 1.27 1.27)
+				)
+				(hide yes)
+			)
+		)
 		(pin "1"
 		)
@@
 		(unit 1)
 		(exclude_from_sim no)
-		(in_bom yes)
+		(in_bom no)
 		(on_board yes)
 		(dnp no)
@@
 		(unit 1)
 		(exclude_from_sim no)
-		(in_bom yes)
+		(in_bom no)
 		(on_board yes)
 		(dnp no)
@@
 			)
 		)
+		(property "PN" "RBR1VWM60ATR "
+			(at 241.3 127 0)
+			(effects
+				(font
+					(size 1.27 1.27)
+				)
+				(hide yes)
+			)
+		)
 		(pin "1"
 		)
@@
 			)
 		)
+		(property "PN" "CB052D0105KBC"
+			(at 208.28 127 0)
+			(effects
+				(font
+					(size 1.27 1.27)
+				)
+				(hide yes)
+			)
+		)
 		(pin "1"
 		)
@@
 			)
 		)
+		(property "PN" "CB052D0105KBC"
+			(at 208.28 80.01 0)
+			(effects
+				(font
+					(size 1.27 1.27)
+				)
+				(hide yes)
+			)
+		)
 		(pin "1"
 		)
@@
 		(unit 1)
 		(exclude_from_sim no)
-		(in_bom yes)
+		(in_bom no)
 		(on_board yes)
 		(dnp no)
@@
 		(unit 1)
 		(exclude_from_sim no)
-		(in_bom yes)
+		(in_bom no)
 		(on_board yes)
 		(dnp no)
@@
 		(unit 1)
 		(exclude_from_sim no)
-		(in_bom yes)
+		(in_bom no)
 		(on_board yes)
 		(dnp no)
@@
 			)
 		)
+		(property "PN" "RBR1VWM60ATR "
+			(at 233.68 96.52 0)
+			(effects
+				(font
+					(size 1.27 1.27)
+				)
+				(hide yes)
+			)
+		)
 		(pin "1"
 		)
@@
 			)
 		)
+		(property "PN" "TPA3255DDVR"
+			(at 111.76 125.73 0)
+			(effects
+				(font
+					(size 1.27 1.27)
+				)
+				(hide yes)
+			)
+		)
 		(pin "1"
 		)
@@
 			)
 		)
+		(property "PN" "RBR1VWM60ATR "
+			(at 233.68 127 0)
+			(effects
+				(font
+					(size 1.27 1.27)
+				)
+				(hide yes)
+			)
+		)
 		(pin "1"
 		)
@@
 			)
 		)
+		(property "PN" "SPM12565VT-100M-D"
+			(at 200.66 92.71 0)
+			(effects
+				(font
+					(size 1.27 1.27)
+				)
+				(hide yes)
+			)
+		)
 		(pin "1"
 		)
@@
 		(unit 1)
 		(exclude_from_sim no)
-		(in_bom yes)
+		(in_bom no)
 		(on_board yes)
 		(dnp no)
@@
 			)
 		)
+		(property "PN" "RBR1VWM60ATR "
+			(at 241.3 114.3 0)
+			(effects
+				(font
+					(size 1.27 1.27)
+				)
+				(hide yes)
+			)
+		)
 		(pin "1"
 		)
@@
 			)
 		)
-		(property "Value" "10nF"
+		(property "Value" "10nF 63V"
 			(at 219.71 128.905 0)
 			(effects
@@
 			)
 		)
+		(property "PN" "C0603X103K2RECTU"
+			(at 215.9 127 0)
+			(effects
+				(font
+					(size 1.27 1.27)
+				)
+				(hide yes)
+			)
+		)
 		(pin "1"
 		)
@@
 		(unit 1)
 		(exclude_from_sim no)
-		(in_bom yes)
+		(in_bom no)
 		(on_board yes)
 		(dnp no)
@@
 			)
 		)
-		(property "Value" "10nF"
+		(property "Value" "10nF 63V"
 			(at 219.71 98.425 0)
 			(effects
@@
 			)
 		)
+		(property "PN" "C0603X103K2RECTU"
+			(at 215.9 96.52 0)
+			(effects
+				(font
+					(size 1.27 1.27)
+				)
+				(hide yes)
+			)
+		)
 		(pin "1"
 		)
@@
 			)
 		)
+		(property "PN" "SPM12565VT-100M-D"
+			(at 200.66 123.19 0)
+			(effects
+				(font
+					(size 1.27 1.27)
+				)
+				(hide yes)
+			)
+		)
 		(pin "1"
 		)
@@
 		(unit 1)
 		(exclude_from_sim no)
-		(in_bom yes)
+		(in_bom no)
 		(on_board yes)
 		(dnp no)
@@
 			)
 		)
-		(property "Value" "10nF"
+		(property "Value" "10nF 63V"
 			(at 219.71 81.915 0)
 			(effects
@@
 			)
 		)
+		(property "PN" "C0603X103K2RECTU"
+			(at 215.9 80.01 0)
+			(effects
+				(font
+					(size 1.27 1.27)
+				)
+				(hide yes)
+			)
+		)
 		(pin "1"
 		)
@@
 			)
 		)
+		(property "PN" "RBR1VWM60ATR "
+			(at 241.3 80.01 0)
+			(effects
+				(font
+					(size 1.27 1.27)
+				)
+				(hide yes)
+			)
+		)
 		(pin "1"
 		)
@@
 			)
 		)
+		(property "PN" "TC33X-2-103E"
+			(at 118.11 180.34 0)
+			(effects
+				(font
+					(size 1.27 1.27)
+				)
+				(hide yes)
+			)
+		)
 		(pin "1"
 		)
@@
 			)
 		)
+		(property "PN" "RBR1VWM60ATR "
+			(at 233.68 80.01 0)
+			(effects
+				(font
+					(size 1.27 1.27)
+				)
+				(hide yes)
+			)
+		)
 		(pin "1"
 		)
@@
 			)
 		)
+		(property "PN" "SPM12565VT-100M-D"
+			(at 200.66 76.2 0)
+			(effects
+				(font
+					(size 1.27 1.27)
+				)
+				(hide yes)
+			)
+		)
 		(pin "1"
 		)
@@
 			)
 		)
+		(property "PN" "SPM12565VT-100M-D"
+			(at 200.66 110.49 0)
+			(effects
+				(font
+					(size 1.27 1.27)
+				)
+				(hide yes)
+			)
+		)
 		(pin "1"
 		)
@@
 			)
 		)
+		(property "PN" "CB052D0105KBC"
+			(at 208.28 96.52 0)
+			(effects
+				(font
+					(size 1.27 1.27)
+				)
+				(hide yes)
+			)
+		)
 		(pin "1"
 		)
@@
 			)
 		)
-		(property "Value" "10nF"
+		(property "Value" "10nF 63V"
 			(at 219.71 116.205 0)
 			(effects
@@
 			(at 215.9 114.3 0)
 			(effects
+				(font
+					(size 1.27 1.27)
+				)
+				(hide yes)
+			)
+		)
+		(property "PN" "C0603X103K2RECTU"
+			(at 215.9 114.3 0)
+			(effects
