File: preamp.kicad_sch (KiCad schematic)
At the start: 17 parts, among them U4 Opamp_Dual

Commit message: fill in some part numbers
Parts:
- R53, R58: value R_Small -> 3.6k; PN (none) -> RT0603DRD073K6L
- R54, R55, R56, R57, R59, R60, R61, R62: PN (none) -> RT0603DRD073K6L
- U4: PN (none) -> NE5532DR
- s2, s3: now left out of the parts list
Changed lines of the file:
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@@
+			)
+		)
+		(property "PN" "NE5532DR"
+			(at 111.76 92.71 0)
+			(effects
+				(font
+					(size 1.27 1.27)
+				)
+				(hide yes)
 			)
 		)
@@
 			)
 		)
+		(property "PN" "RT0603DRD073K6L"
+			(at 38.1 80.01 0)
+			(effects
+				(font
+					(size 1.27 1.27)
+				)
+				(hide yes)
+			)
+		)
 		(pin "1"
 		)
@@
 			)
 		)
+		(property "PN" "RT0603DRD073K6L"
+			(at 38.1 72.39 0)
+			(effects
+				(font
+					(size 1.27 1.27)
+				)
+				(hide yes)
+			)
+		)
 		(pin "1"
 		)
@@
 			)
 		)
+		(property "PN" "RT0603DRD073K6L"
+			(at 38.1 64.77 0)
+			(effects
+				(font
+					(size 1.27 1.27)
+				)
+				(hide yes)
+			)
+		)
 		(pin "1"
 		)
@@
 			)
 		)
+		(property "PN" "NE5532DR"
+			(at 58.42 46.99 0)
+			(effects
+				(font
+					(size 1.27 1.27)
+				)
+				(hide yes)
+			)
+		)
 		(pin "1"
 		)
@@
 			)
 		)
+		(property "PN" "RT0603DRD073K6L"
+			(at 38.1 130.81 0)
+			(effects
+				(font
+					(size 1.27 1.27)
+				)
+				(hide yes)
+			)
+		)
 		(pin "1"
 		)
@@
 			)
 		)
+		(property "PN" "RT0603DRD073K6L"
+			(at 38.1 138.43 0)
+			(effects
+				(font
+					(size 1.27 1.27)
+				)
+				(hide yes)
+			)
+		)
 		(pin "1"
 		)
@@
 			)
 		)
+		(property "PN" "RT0603DRD073K6L"
+			(at 38.1 115.57 0)
+			(effects
+				(font
+					(size 1.27 1.27)
+				)
+				(hide yes)
+			)
+		)
 		(pin "1"
 		)
@@
 			)
 		)
-		(property "Value" "R_Small"
+		(property "Value" "3.6k"
 			(at 38.1 46.99 90)
 			(effects
@@
 		)
 		(property "Sim.Pins" ""
+			(at 38.1 49.53 0)
+			(effects
+				(font
+					(size 1.27 1.27)
+				)
+				(hide yes)
+			)
+		)
+		(property "PN" "RT0603DRD073K6L"
 			(at 38.1 49.53 0)
 			(effects
@@
 			)
 		)
+		(property "PN" "RT0603DRD073K6L"
+			(at 38.1 57.15 0)
+			(effects
+				(font
+					(size 1.27 1.27)
+				)
+				(hide yes)
+			)
+		)
 		(pin "1"
 		)
@@
 		(unit 1)
 		(exclude_from_sim no)
-		(in_bom yes)
+		(in_bom no)
 		(on_board yes)
 		(dnp no)
@@
 			)
 		)
+		(property "PN" "NE5532DR"
+			(at 58.42 105.41 0)
+			(effects
+				(font
+					(size 1.27 1.27)
+				)
+				(hide yes)
+			)
+		)
 		(pin "1"
 		)
@@
 		(unit 1)
 		(exclude_from_sim no)
-		(in_bom yes)
+		(in_bom no)
 		(on_board yes)
 		(dnp no)
@@
 			)
 		)
+		(property "PN" "RT0603DRD073K6L"
+			(at 38.1 123.19 0)
+			(effects
+				(font
+					(size 1.27 1.27)
+				)
+				(hide yes)
+			)
+		)
 		(pin "1"
 		)
@@
 			)
 		)
-		(property "Value" "R_Small"
+		(property "Value" "3.6k"
 			(at 38.1 105.41 90)
 			(effects
@@
 			(at 38.1 107.95 0)
 			(effects
+				(font
+					(size 1.27 1.27)
+				)
+				(hide yes)
+			)
+		)
+		(property "PN" "RT0603DRD073K6L"
+			(at 38.1 107.95 0)
+			(effects

Commit message: update partnumbers to what was bought
Parts:
- U4: value Opamp_Dual -> NE5532
Changed lines of the file:
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@@
 			)
 		)
-		(property "Value" "Opamp_Dual"
+		(property "Value" "NE5532"
 			(at 110.49 94.615 0)
 			(effects
@@
 			)
 		)
-		(property "Value" "Opamp_Dual"
+		(property "Value" "NE5532"
 			(at 58.42 40.64 0)
 			(effects
@@
 			)
 		)
-		(property "Value" "Opamp_Dual"
+		(property "Value" "NE5532"
 			(at 58.42 99.06 0)
 			(effects
