File: preamp.kicad_sch (KiCad schematic)
At the start: 17 parts, among them U4 NE5532

Commit message: workaround major gain/signal margin error
using the components i have at hand. There probably are better options. Next revision should make use of the -5v rail.
Parts:
- R53, R54, R55, R56, R57, R58, R59, R60, R61, R62: value 3.6k -> t2k
- R63, R64: value 2k -> t2k
- U4: value NE5532 -> OPA1642; PN NE5532DR -> (none)
Other:
- note added: "up to 6.9vpp use: 4.76vpp"
- note removed: "up to 9vpp"
Changed lines of the file:
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@@
 		)
 	)
-	(text "up to 9vpp"
+	(text "up to 6.9vpp\nuse: 4.76vpp"
 		(exclude_from_sim no)
-		(at 19.05 60.96 0)
+		(at 17.272 62.992 0)
 		(effects
 			(font
@@
 			)
 		)
-		(property "Value" "NE5532"
+		(property "Value" "OPA1642"
 			(at 110.49 94.615 0)
 			(effects
@@
 			)
 		)
-		(property "PN" "NE5532DR"
+		(property "PN" ""
 			(at 111.76 92.71 0)
 			(effects
@@
 			)
 		)
-		(property "Value" "3.6k"
+		(property "Value" "t2k"
 			(at 38.1 77.47 90)
 			(effects
@@
 			)
 		)
-		(property "Value" "3.6k"
+		(property "Value" "t2k"
 			(at 38.1 69.85 90)
 			(effects
@@
 			)
 		)
-		(property "Value" "3.6k"
+		(property "Value" "t2k"
 			(at 38.1 62.23 90)
 			(effects
@@
 			)
 		)
-		(property "Value" "NE5532"
+		(property "Value" "OPA1642"
 			(at 58.42 40.64 0)
 			(effects
@@
 			)
 		)
-		(property "PN" "NE5532DR"
+		(property "PN" ""
 			(at 58.42 46.99 0)
 			(effects
@@
 			)
 		)
-		(property "Value" "3.6k"
+		(property "Value" "t2k"
 			(at 38.1 128.27 90)
 			(effects
@@
 			)
 		)
-		(property "Value" "3.6k"
+		(property "Value" "t2k"
 			(at 38.1 135.89 90)
 			(effects
@@
 			)
 		)
-		(property "Value" "3.6k"
+		(property "Value" "t2k"
 			(at 38.1 113.03 90)
 			(effects
@@
 			)
 		)
-		(property "Value" "3.6k"
+		(property "Value" "t2k"
 			(at 38.1 46.99 90)
 			(effects
@@
 			)
 		)
-		(property "Value" "2k"
+		(property "Value" "t2k"
 			(at 58.42 114.3 90)
 			(effects
@@
 			)
 		)
-		(property "Value" "3.6k"
+		(property "Value" "t2k"
 			(at 38.1 54.61 90)
 			(effects
@@
 			)
 		)
-		(property "Value" "2k"
+		(property "Value" "t2k"
 			(at 58.42 55.88 90)
 			(effects
@@
 			)
 		)
-		(property "Value" "NE5532"
+		(property "Value" "OPA1642"
 			(at 58.42 99.06 0)
 			(effects
@@
 			)
 		)
-		(property "PN" "NE5532DR"
+		(property "PN" ""
 			(at 58.42 105.41 0)
 			(effects
@@
 			)
 		)
-		(property "Value" "3.6k"
+		(property "Value" "t2k"
 			(at 38.1 120.65 90)
 			(effects
@@
 			)
 		)
-		(property "Value" "3.6k"
+		(property "Value" "t2k"
 			(at 38.1 105.41 90)
 			(effects

Commit message: work on bugs...
Parts:
- U4: value OPA1642 -> MC33078; PN (none) -> MC33078
Changed lines of the file:
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@@
 			)
 		)
-		(property "Value" "OPA1642"
+		(property "Value" "MC33078"
 			(at 110.49 94.615 0)
 			(effects
@@
 			)
 		)
-		(property "PN" ""
+		(property "PN" "MC33078"
 			(at 111.76 92.71 0)
 			(effects
@@
 			)
 		)
-		(property "Value" "OPA1642"
+		(property "Value" "MC33078"
 			(at 58.42 40.64 0)
 			(effects
@@
 			)
 		)
-		(property "PN" ""
+		(property "PN" "MC33078"
 			(at 58.42 46.99 0)
 			(effects
@@
 			)
 		)
-		(property "Value" "OPA1642"
+		(property "Value" "MC33078"
 			(at 58.42 99.06 0)
 			(effects
@@
 			)
 		)
-		(property "PN" ""
+		(property "PN" "MC33078"
 			(at 58.42 105.41 0)
 			(effects

Commit message: work on bugs
* align parts
* enlarge cercaps
* fix ak caps
* improve jack footprint
* fix lmr stencil openings
* remove one ldo
Parts:
- CRP1, CU4: footprint invendelirium_audio:C_0603 -> invendelirium_audio:C_0603_larger
Changed lines of the file:
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@@
 			)
 		)
-		(property "Footprint" "invendelirium_audio:C_0603"
+		(property "Footprint" "invendelirium_audio:C_0603_larger"
 			(at 126.6952 97.79 0)
 			(effects
@@
 			)
 		)
-		(property "Footprint" "invendelirium_audio:C_0603"
+		(property "Footprint" "invendelirium_audio:C_0603_larger"
 			(at 54.3052 82.55 0)
 			(effects

Commit message: more bom updates
Parts:
- R55, R59: now not fitted
Changed lines of the file:
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@@
 		(in_bom yes)
 		(on_board yes)
-		(dnp no)
+		(dnp yes)
 		(fields_autoplaced yes)
 		(property "Reference" "R55"
@@
 		(in_bom yes)
 		(on_board yes)
-		(dnp no)
+		(dnp yes)
 		(fields_autoplaced yes)
 		(property "Reference" "R59"
