File: dac_amp.kicad_sch (KiCad schematic)
At the start: 21 parts, among them U16 MC33078

Commit message: work on bugs
* align parts
* enlarge cercaps
* fix ak caps
* improve jack footprint
* fix lmr stencil openings
* remove one ldo
Parts:
- CRD2, CU15: footprint invendelirium_audio:C_0603 -> invendelirium_audio:C_0603_larger
Changed lines of the file:
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@@
 			)
 		)
-		(property "Footprint" "invendelirium_audio:C_0603"
+		(property "Footprint" "invendelirium_audio:C_0603_larger"
 			(at 74.6252 138.43 0)
 			(effects
@@
 			)
 		)
-		(property "Footprint" "invendelirium_audio:C_0603"
+		(property "Footprint" "invendelirium_audio:C_0603_larger"
 			(at 89.8652 137.16 0)
 			(effects
