File: dac-supply.kicad_sch (KiCad schematic)
At the start: 5 parts, among them U10 L78L05_SOT89

Commit message: work on bugs
Parts:
- U10: footprint Package_TO_SOT_SMD:SOT-89-3 -> invendelirium_general:SOT-89-3
Changed lines of the file:
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@@
 			)
 		)
-		(property "Footprint" "Package_TO_SOT_SMD:SOT-89-3"
+		(property "Footprint" "invendelirium_general:SOT-89-3"
 			(at 69.85 33.02 0)
 			(effects
