File: feedbass_preamp.kicad_sch (KiCad schematic)
At the start: 15 parts, among them J2 Conn_Coaxial, U7 Opamp_Dual

Commit message: some routing till got stuck
got stuck on U16's power part somehow being on a different sheet
Parts:
- C72: PN (none) -> FCA1206C334M-H2
Changed lines of the file:
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@@
+			)
+		)
+		(property "PN" "FCA1206C334M-H2"
+			(at 153.67 54.61 90)
+			(effects
+				(font
+					(size 1.016 1.016)
+				)
+				(hide yes)
 			)
 		)

Commit message: update some footprints
Parts:
- D17: footprint Diode_SMD:D_SOD-323_HandSoldering -> invendelirium_general:D_SOD-323
Changed lines of the file:
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@@
 			)
 		)
-		(property "Footprint" "Diode_SMD:D_SOD-323_HandSoldering"
+		(property "Footprint" "invendelirium_general:D_SOD-323"
 			(at 66.04 67.31 0)
 			(effects

Commit message: fill in some part numbers
Parts:
- RV3: PN (none) -> PV37X102C01B00
- U7: PN (none) -> OPA1642AIDGKR
Changed lines of the file:
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@@
+			)
+		)
+		(property "PN" "OPA1642AIDGKR"
+			(at 181.61 72.39 0)
+			(effects
+				(font
+					(size 1.27 1.27)
+				)
+				(hide yes)
 			)
 		)
@@
 			)
 		)
+		(property "PN" "OPA1642AIDGKR"
+			(at 133.35 49.53 0)
+			(effects
+				(font
+					(size 1.27 1.27)
+				)
+				(hide yes)
+			)
+		)
 		(pin "1"
 		)
@@
 			)
 		)
+		(property "PN" "OPA1642AIDGKR"
+			(at 137.16 118.11 0)
+			(effects
+				(font
+					(size 1.27 1.27)
+				)
+				(hide yes)
+			)
+		)
 		(pin "1"
 		)
@@
 			(at 119.38 57.15 0)
 			(effects
+				(font
+					(size 1.27 1.27)
+				)
+				(hide yes)
+			)
+		)
+		(property "PN" "PV37X102C01B00"
+			(at 119.38 57.15 0)
+			(effects

Commit message: update partnumbers to what was bought
Parts:
- RV3: PN PV37X102C01B00 -> PV37X202C01B00
- U7: value Opamp_Dual -> OPA1642; PN OPA1642AIDGKR -> OPA1642AIDR
Changed lines of the file:
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@@
 			)
 		)
-		(property "Value" "Opamp_Dual"
+		(property "Value" "OPA1642"
 			(at 181.61 66.04 0)
 			(effects
@@
 			)
 		)
-		(property "PN" "OPA1642AIDGKR"
+		(property "PN" "OPA1642AIDR"
 			(at 181.61 72.39 0)
 			(effects
@@
 			)
 		)
-		(property "Value" "Opamp_Dual"
+		(property "Value" "OPA1642"
 			(at 133.35 43.18 0)
 			(effects
@@
 			)
 		)
-		(property "PN" "OPA1642AIDGKR"
+		(property "PN" "OPA1642AIDR"
 			(at 133.35 49.53 0)
 			(effects
@@
 			)
 		)
-		(property "Value" "Opamp_Dual"
+		(property "Value" "OPA1642"
 			(at 135.89 120.015 0)
 			(effects
@@
 			)
 		)
-		(property "PN" "OPA1642AIDGKR"
+		(property "PN" "OPA1642AIDR"
 			(at 137.16 118.11 0)
 			(effects
@@
 			)
 		)
-		(property "PN" "PV37X102C01B00"
+		(property "PN" "PV37X202C01B00"
 			(at 119.38 57.15 0)
 			(effects

Commit message: workaround major gain/signal margin error
using the components i have at hand. There probably are better options. Next revision should make use of the -5v rail.
Parts:
- R71, R72: value 2k -> t2k
- RV3: value 1k -> 2k
Changed lines of the file:
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@@
 			)
 		)
-		(property "Value" "2k"
+		(property "Value" "t2k"
 			(at 181.61 80.01 90)
 			(effects
@@
 			)
 		)
-		(property "Value" "1k"
+		(property "Value" "2k"
 			(at 116.84 55.245 0)
 			(effects
@@
 			)
 		)
-		(property "Value" "2k"
+		(property "Value" "t2k"
 			(at 161.29 72.39 90)
 			(effects

Commit message: work on bugs
* align parts
* enlarge cercaps
* fix ak caps
* improve jack footprint
* fix lmr stencil openings
* remove one ldo
Parts:
- CRB0, CU7: footprint invendelirium_audio:C_0603 -> invendelirium_audio:C_0603_larger
Changed lines of the file:
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@@
 			)
 		)
-		(property "Footprint" "invendelirium_audio:C_0603"
+		(property "Footprint" "invendelirium_audio:C_0603_larger"
 			(at 134.3152 88.9 0)
 			(effects
@@
 			)
 		)
-		(property "Footprint" "invendelirium_audio:C_0603"
+		(property "Footprint" "invendelirium_audio:C_0603_larger"
 			(at 153.3652 123.19 0)
 			(effects

Commit message: reroute feedbass amps
+ add the missing discharge resistor
Parts:
- added R241: 47M, invendelirium_audio:R_0603, symbol Device:R_Small
- C69, C70: footprint Capacitor_SMD:C_0805_2012Metric -> invendelirium_general:C_0805
Connections:
- net fakegnd: now also RV3.1, R241.1; no longer RV3.3
- net at C69.1, J2.1 (In), R73.1: now also R241.2
- net at R74.1, U7.1: now also RV3.3; no longer RV3.1
Changed lines of the file:
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@@
 	(paper "A4")
+	(junction
+		(at 82.55 54.61)
+		(diameter 0)
+		(color 0 0 0 0)
+	)
 	(junction
 		(at 82.55 46.99)
@@
 	)
 	(junction
+		(at 71.12 46.99)
+		(diameter 0)
+		(color 0 0 0 0)
+	)
+	(junction
 		(at 116.84 62.23)
 		(diameter 0)
@@
 	(wire
 		(pts
+			(xy 71.12 54.61) (xy 82.55 54.61)
+		)
+		(stroke
+			(width 0)
+			(type default)
+		)
+	)
+	(wire
+		(pts
 			(xy 168.91 69.85) (xy 168.91 72.39)
 		)
@@
 	(wire
 		(pts
+			(xy 71.12 53.34) (xy 71.12 54.61)
+		)
+		(stroke
+			(width 0)
+			(type default)
+		)
+	)
+	(wire
+		(pts
 			(xy 184.15 82.55) (xy 190.5 82.55)
 		)
@@
 	(wire
 		(pts
+			(xy 71.12 46.99) (xy 82.55 46.99)
+		)
+		(stroke
+			(width 0)
+			(type default)
+		)
+	)
+	(wire
+		(pts
 			(xy 156.21 74.93) (xy 156.21 66.04)
 		)
@@
 	(wire
 		(pts
-			(xy 67.31 46.99) (xy 82.55 46.99)
+			(xy 67.31 46.99) (xy 71.12 46.99)
 		)
 		(stroke
@@
 		(pts
 			(xy 142.24 49.53) (xy 140.97 49.53)
+		)
+		(stroke
+			(width 0)
+			(type default)
+		)
+	)
+	(wire
+		(pts
+			(xy 71.12 46.99) (xy 71.12 48.26)
 		)
 		(stroke
@@
 			)
 		)
-		(property "Footprint" "Capacitor_SMD:C_0805_2012Metric"
+		(property "Footprint" "invendelirium_general:C_0805"
 			(at 105.1052 54.61 0)
 			(effects
@@
 	)
 	(symbol
+		(lib_id "Device:R_Small")
+		(at 71.12 50.8 180)
+		(unit 1)
+		(exclude_from_sim no)
+		(in_bom yes)
+		(on_board yes)
+		(dnp no)
+		(fields_autoplaced yes)
+		(property "Reference" "R241"
+			(at 73.66 49.5299 0)
+			(effects
+				(font
+					(size 1.27 1.27)
+				)
+				(justify right)
+			)
+		)
+		(property "Value" "47M"
+			(at 73.66 52.0699 0)
+			(effects
+				(font
+					(size 1.27 1.27)
+				)
+				(justify right)
+			)
+		)
+		(property "Footprint" "invendelirium_audio:R_0603"
+			(at 71.12 50.8 0)
+			(effects
+				(font
+					(size 1.27 1.27)
+				)
+				(hide yes)
+			)
+		)
+		(property "Datasheet" "~"
+			(at 71.12 50.8 0)
+			(effects
+				(font
+					(size 1.27 1.27)
+				)
+				(hide yes)
+			)
+		)
+		(property "Description" ""
+			(at 71.12 50.8 0)
+			(effects
+				(font
+					(size 1.27 1.27)
+				)
+				(hide yes)
+			)
+		)
+		(property "Sim.Device" ""
+			(at 71.12 50.8 0)
+			(effects
+				(font
+					(size 1.27 1.27)
+				)
+				(hide yes)
+			)
+		)
+		(property "Sim.Library" ""
+			(at 71.12 50.8 0)
+			(effects
+				(font
+					(size 1.27 1.27)
+				)
+				(hide yes)
+			)
+		)
+		(property "Sim.Name" ""
+			(at 71.12 50.8 0)
+			(effects
+				(font
+					(size 1.27 1.27)
+				)
+				(hide yes)
+			)
+		)
+		(property "Sim.Pins" ""
+			(at 71.12 50.8 0)
+			(effects
+				(font
+					(size 1.27 1.27)
+				)
+				(hide yes)
+			)
+		)
+		(pin "1"
+		)
+		(pin "2"
+		)
+		(instances
+			(project "uberamp1"
+				(path "/310059c1-d84b-43e2-9c9a-0e426c534a12/605c496f-1ba6-4b8d-86f6-e928e6401a1d"
+					(reference "R241")
+					(unit 1)
+				)
+				(path "/310059c1-d84b-43e2-9c9a-0e426c534a12/fb6b8bc8-ff14-4d64-816d-20c0f51b1294"
+					(reference "R242")
+					(unit 1)
+				)
+			)
+		)
+	)
+	(symbol
 		(lib_id "Device:C")
 		(at 133.35 85.09 0)
@@
 			)
 		)
-		(property "Footprint" "Capacitor_SMD:C_0805_2012Metric"
+		(property "Footprint" "invendelirium_general:C_0805"
 			(at 83.5152 54.61 0)
 			(effects
@@
 		(lib_id "Device:R_Potentiometer_Small")
 		(at 119.38 57.15 0)
-		(mirror x)
 		(unit 1)
 		(exclude_from_sim no)
@@
 		(dnp no)
 		(property "Reference" "RV3"
-			(at 116.84 57.785 0)
+			(at 116.84 56.515 0)
 			(effects
 				(font
@@
 		)
 		(property "Value" "2k"
-			(at 116.84 55.245 0)
-			(effects
-				(font
+			(at 116.84 59.055 0)
+			(effects
+				(font

Commit message: work on bugs
Parts:
- C72: footprint Capacitor_SMD:C_1206_3216Metric -> invendelirium_general:C_1206
Changed lines of the file:
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@@
 			)
 		)
-		(property "Footprint" "Capacitor_SMD:C_1206_3216Metric"
+		(property "Footprint" "invendelirium_general:C_1206"
 			(at 154.6352 58.42 0)
 			(effects
