File: dsp.kicad_sch (KiCad schematic)
At the start: 56 parts, among them J3 pots, J4 Conn_01x04, Q1 Q_PNP_BCE, U15 Opamp_Dual, U22 ADAU1701, U23 MC33275, U24 MC33275, U30 M24128 (128kbit)

Commit message: update partnumbers to what was bought
Parts:
- U15: value Opamp_Dual -> OPA2322
Changed lines of the file:
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@@
 			)
 		)
-		(property "Value" "Opamp_Dual"
+		(property "Value" "OPA2322"
 			(at 205.74 60.325 0)
 			(effects
@@
 			)
 		)
-		(property "Value" "Opamp_Dual"
+		(property "Value" "OPA2322"
 			(at 90.17 146.05 0)
 			(effects
@@
 			)
 		)
-		(property "Value" "Opamp_Dual"
+		(property "Value" "OPA2322"
 			(at 214.63 71.12 0)
 			(effects

Commit message: update values to what's being used + mark thin film resistors
Parts:
- R190: value 18k -> t18k
Changed lines of the file:
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@@
 			)
 		)
-		(property "Value" "18k"
+		(property "Value" "t18k"
 			(at 107.95 71.12 90)
 			(effects

Commit message: work on bugs
* align parts
* enlarge cercaps
* fix ak caps
* improve jack footprint
* fix lmr stencil openings
* remove one ldo
Parts:
- removed U23: MC33275, invendelirium_general:SOT-223-3_TabPin2, symbol Regulator_Linear:L7805
- C133, C136, C137, C141, C143, C78, C82, CU16, CU22, CU23, CU30: footprint invendelirium_audio:C_0603 -> invendelirium_audio:C_0603_larger
Other:
- moved on the sheet: J4

Commit message: work on bugs
Parts:
- added R218, R219: 10k, invendelirium_audio:R_0603, symbol Device:R_Small
- J4: footprint Connector_PinHeader_2.54mm:PinHeader_1x04_P2.54mm_Vertical -> Connector_JST:JST_GH_BM04B-GHS-TBT_1x04-1MP_P1.25mm_Vertical
Connections:
- net +3v3_d: now also R218.2, R219.2
- net GND: now also J4.4 (Pin_4); no longer J4.1 (Pin_1)
- net i2c_scl: now also J4.2 (Pin_2), R219.1; no longer J4.3 (Pin_3)
- net i2c_sda: now also J4.3 (Pin_3), R218.1; no longer J4.2 (Pin_2)
Other:
- note added: "vcc scl sda gnd"

Commit message: all known bugs fixed
Parts:
- J4: now not fitted
Other:
- sheet audio_input ports: added -5V; removed none
- sheet line_out ports: added -5V; removed none
Changed lines of the file:
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@@
 	)
 	(junction
+		(at 281.94 33.02)
+		(diameter 0)
+		(color 0 0 0 0)
+	)
+	(junction
 		(at 194.31 74.93)
 		(diameter 0)
@@
 	)
 	(junction
+		(at 57.15 36.83)
+		(diameter 0)
+		(color 0 0 0 0)
+	)
+	(junction
 		(at 233.68 80.01)
 		(diameter 0)
@@
 	(wire
 		(pts
+			(xy 57.15 36.83) (xy 59.69 36.83)
+		)
+		(stroke
+			(width 0)
+			(type default)
+		)
+	)
+	(wire
+		(pts
 			(xy 110.49 73.66) (xy 113.03 73.66)
 		)
@@
 	(wire
 		(pts
+			(xy 57.15 36.83) (xy 57.15 40.64)
+		)
+		(stroke
+			(width 0)
+			(type default)
+		)
+	)
+	(wire
+		(pts
 			(xy 154.94 88.9) (xy 156.21 88.9)
 		)
@@
 	(wire
 		(pts
+			(xy 281.94 33.02) (xy 284.48 33.02)
+		)
+		(stroke
+			(width 0)
+			(type default)
+		)
+	)
+	(wire
+		(pts
 			(xy 248.92 60.96) (xy 251.46 60.96)
 		)
@@
 	(wire
 		(pts
+			(xy 280.67 33.02) (xy 281.94 33.02)
+		)
+		(stroke
+			(width 0)
+			(type default)
+		)
+	)
+	(wire
+		(pts
 			(xy 156.21 46.99) (xy 146.05 46.99)
 		)
@@
 	(wire
 		(pts
+			(xy 280.67 41.91) (xy 281.94 41.91)
+		)
+		(stroke
+			(width 0)
+			(type default)
+		)
+	)
+	(wire
+		(pts
 			(xy 186.69 99.06) (xy 213.36 99.06)
 		)
@@
 	(wire
 		(pts
+			(xy 55.88 36.83) (xy 57.15 36.83)
+		)
+		(stroke
+			(width 0)
+			(type default)
+		)
+	)
+	(wire
+		(pts
 			(xy 135.89 124.46) (xy 138.43 124.46)
 		)
@@
 	(wire
 		(pts
+			(xy 281.94 41.91) (xy 281.94 33.02)
+		)
+		(stroke
+			(width 0)
+			(type default)
+		)
+	)
+	(wire
+		(pts
 			(xy 43.18 68.58) (xy 54.61 68.58)
 		)
@@
 		)
 	)
+	(label "-5V"
+		(at 55.88 36.83 0)
+		(fields_autoplaced yes)
+		(effects
+			(font
+				(size 1.016 1.016)
+			)
+			(justify left bottom)
+		)
+	)
 	(label "aux1"
 		(at 101.6 165.1 0)
@@
 		)
 	)
+	(label "-5V"
+		(at 280.67 33.02 0)
+		(fields_autoplaced yes)
+		(effects
+			(font
+				(size 1.016 1.016)
+			)
+			(justify left bottom)
+		)
+	)
 	(label "aux3"
 		(at 166.37 106.68 0)
@@
 		(in_bom yes)
 		(on_board yes)
-		(dnp no)
+		(dnp yes)
 		(property "Reference" "J4"
 			(at 19.812 134.112 0)
@@
 			)
 		)
+		(pin "-5V" output
+			(at 280.67 41.91 0)
+			(effects
+				(font
+					(size 1.016 1.016)
+				)
+				(justify right)
+			)
+		)
 		(instances
 			(project "uberamp1"
@@
 			(effects
 				(font
+					(size 1.016 1.016)
+				)
+				(justify right)
+			)
+		)
+		(pin "-5V" input
+			(at 57.15 40.64 90)
+			(effects
+				(font

Commit message: fix connector part number
Parts:
- J3: PN BM03B-GHS-TBT -> BM06B-GHS-TBT
Changed lines of the file:
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@@
 			)
 		)
-		(property "PN" "BM03B-GHS-TBT"
+		(property "PN" "BM06B-GHS-TBT"
 			(at 22.86 165.1 0)
 			(effects
